Commit message: Added IMU

File: ros2_ws/src/robot_description/urdf/gazebo_setup.xacro (robot description, xacro)
@@ -24,4 +24,5 @@
     <gazebo reference="lidar_link">
         <sensor name="lidar_sensor" type="gpu_lidar">
+            <frame_name>lidar_link</frame_name>
             <topic>scan</topic>
             <update_rate>10</update_rate>
@@ -54,4 +55,61 @@
     </gazebo>
     <gazebo>
+        <plugin name='gz::sim::systems::Imu' filename='gz-sim-imu-system'/>
+    </gazebo>
+    <gazebo reference="imu_link">
+        <sensor name="imu" type="imu">
+            <always_on>true</always_on>
+            <update_rate>100</update_rate>
+            <gz_frame_id>imu_link</gz_frame_id>
+            <topic>imu</topic>
+            <!-- <visualize>true</visualize>
+            <frame>
+                <pose relative_to="imu_link">0 0 0 0 0 0</pose>
+            </frame> -->
+            <imu>
+                <angular_velocity>
+                    <x>
+                        <noise type="gaussian">
+                            <mean>0.0</mean>
+                            <stddev>2e-4</stddev>
+                        </noise>
+                    </x>
+                    <y>
+                        <noise type="gaussian">
+                            <mean>0.0</mean>
+                            <stddev>2e-4</stddev>
+                        </noise>
+                    </y>
+                    <z>
+                        <noise type="gaussian">
+                            <mean>0.0</mean>
+                            <stddev>2e-4</stddev>
+                        </noise>
+                    </z>
+                </angular_velocity>
+                <linear_acceleration>
+                    <x>
+                        <noise type="gaussian">
+                            <mean>0.0</mean>
+                            <stddev>1.7e-2</stddev>
+                        </noise>
+                    </x>
+                    <y>
+                        <noise type="gaussian">
+                            <mean>0.0</mean>
+                            <stddev>1.7e-2</stddev>
+                        </noise>
+                    </y>
+                    <z>
+                        <noise type="gaussian">
+                            <mean>0.0</mean>
+                            <stddev>1.7e-2</stddev>
+                        </noise>
+                    </z>
+                </linear_acceleration>
+            </imu>
+        </sensor>
+    </gazebo>
+    <gazebo>
         <plugin filename="libgz_ros2_control-system.so" name="gz_ros2_control::GazeboSimROS2ControlPlugin">
             <parameters>$(find robot_bringup)/config/controllers.yaml</parameters>

File: ros2_ws/src/robot_description/urdf/properties.xacro (robot description, xacro)
@@ -15,4 +15,7 @@
     <xacro:property name="lidar_radius"     value="0.04"/>
     <xacro:property name="lidar_height"     value="0.1"/>
+    <!-- IMU -->
+    <xacro:property name="imu_length" value="0.04"/>
+    <xacro:property name="imu_height" value="0.01"/>
     <!-- Mass values (kg) -->
     <xacro:property name="chassis_mass"     value="3"/>

File: ros2_ws/src/robot_description/urdf/robot_description.urdf.xacro (robot description, xacro)
@@ -118,4 +118,6 @@
     <!-- LiDAR -->
     <xacro:include filename="$(find robot_description)/urdf/lidar.xacro" />
+    <!-- IMU -->
+    <xacro:include filename="$(find robot_description)/urdf/imu.xacro" />
     <!-- GAZEBO SETUP: Plugin Configuration -->
     <xacro:include filename="$(find robot_description)/urdf/gazebo_setup.xacro" />
